Commit message: made name chanege of package

File: src/description/urdf/basic_terrain_v2_Landscape_01.urdf.xacro (robot description, xacro)
@@ -12,5 +12,5 @@
       <origin xyz="0 0 0" rpy="0 0 0" />
       <geometry>
-        <mesh filename="file://$(find custom_gazebo)/src/description/meshes/basic_terrain_v2_Landscape_01.dae" />
+        <mesh filename="file://$(find custom_gazebo_world)/src/description/meshes/basic_terrain_v2_Landscape_01.dae" />
       </geometry>
     </visual>
@@ -18,5 +18,5 @@
       <origin xyz="0 0 0" rpy="0 0 0" />
       <geometry>
-        <mesh filename="package://custom_gazebo/src/description/meshes/basic_terrain_v2_Landscape_01.dae" />
+        <mesh filename="package://custom_gazebo_world/src/description/meshes/basic_terrain_v2_Landscape_01.dae" />
       </geometry>
     </collision> -->

File: src/description/urdf/basic_terrain_v2_Plane.urdf.xacro (robot description, xacro)
@@ -10,5 +10,5 @@
       <origin xyz="0 0 0" rpy="0 0 0" />
       <geometry>
-        <mesh filename="file://$(find custom_gazebo)/src/description/meshes/basic_terrain_v2_Plane.dae" />
+        <mesh filename="file://$(find custom_gazebo_world)/src/description/meshes/basic_terrain_v2_Plane.dae" />
       </geometry>
     </visual>
@@ -16,5 +16,5 @@
       <origin xyz="0 0 0" rpy="0 0 0" />
       <geometry>
-        <mesh filename="file://$(find custom_gazebo)/src/description/meshes/basic_terrain_v2_Plane.dae" />
+        <mesh filename="file://$(find custom_gazebo_world)/src/description/meshes/basic_terrain_v2_Plane.dae" />
       </geometry>
     </collision>

File: src/description/urdf/basic_terrain_v2_leaves.urdf.xacro (robot description, xacro)
@@ -10,5 +10,5 @@
       <origin xyz="0 0 0" rpy="0 0 0" />
       <geometry>
-        <mesh filename="file://$(find custom_gazebo)/src/description/meshes/basic_terrain_v2_leaves.dae" />
+        <mesh filename="file://$(find custom_gazebo_world)/src/description/meshes/basic_terrain_v2_leaves.dae" />
       </geometry>
     </visual>
@@ -16,5 +16,5 @@
       <origin xyz="0 0 0" rpy="0 0 0" />
       <geometry>
-        <mesh filename="file://$(find custom_gazebo)/src/description/meshes/basic_terrain_v2_leaves.dae" />
+        <mesh filename="file://$(find custom_gazebo_world)/src/description/meshes/basic_terrain_v2_leaves.dae" />
       </geometry>
     </collision> -->

File: src/description/urdf/basic_terrain_v2_leaves_001.001.urdf.xacro (robot description, xacro)
@@ -10,5 +10,5 @@
       <origin xyz="0 0 0" rpy="0 0 0" />
       <geometry>
-        <mesh filename="file://$(find custom_gazebo)/src/description/meshes/basic_terrain_v2_leaves_001.001.dae" />
+        <mesh filename="file://$(find custom_gazebo_world)/src/description/meshes/basic_terrain_v2_leaves_001.001.dae" />
       </geometry>
     </visual>
@@ -16,5 +16,5 @@
       <origin xyz="0 0 0" rpy="0 0 0" />
       <geometry>
-        <mesh filename="file://$(find custom_gazebo)/src/description/meshes/basic_terrain_v2_leaves_001.001.dae" />
+        <mesh filename="file://$(find custom_gazebo_world)/src/description/meshes/basic_terrain_v2_leaves_001.001.dae" />
       </geometry>
     </collision> -->

File: src/description/urdf/basic_terrain_v2_leaves_001.urdf.xacro (robot description, xacro)
@@ -10,5 +10,5 @@
       <origin xyz="0 0 0" rpy="0 0 0" />
       <geometry>
-        <mesh filename="file://$(find custom_gazebo)/src/description/meshes/basic_terrain_v2_leaves_001.dae" />
+        <mesh filename="file://$(find custom_gazebo_world)/src/description/meshes/basic_terrain_v2_leaves_001.dae" />
       </geometry>
     </visual>
@@ -16,5 +16,5 @@
       <origin xyz="0 0 0" rpy="0 0 0" />
       <geometry>
-        <mesh filename="file://$(find custom_gazebo)/src/description/meshes/basic_terrain_v2_leaves_001.dae" />
+        <mesh filename="file://$(find custom_gazebo_world)/src/description/meshes/basic_terrain_v2_leaves_001.dae" />
       </geometry>
     </collision> -->

File: src/description/urdf/basic_terrain_v2_leaves_001_001.urdf.xacro (robot description, xacro)
@@ -10,5 +10,5 @@
       <origin xyz="0 0 0" rpy="0 0 0" />
       <geometry>
-        <mesh filename="file://$(find custom_gazebo)/src/description/meshes/basic_terrain_v2_leaves_001_001.dae" />
+        <mesh filename="file://$(find custom_gazebo_world)/src/description/meshes/basic_terrain_v2_leaves_001_001.dae" />
       </geometry>
     </visual>
@@ -16,5 +16,5 @@
       <origin xyz="0 0 0" rpy="0 0 0" />
       <geometry>
-        <mesh filename="file://$(find custom_gazebo)/src/description/meshes/basic_terrain_v2_leaves_001_001.dae" />
+        <mesh filename="file://$(find custom_gazebo_world)/src/description/meshes/basic_terrain_v2_leaves_001_001.dae" />
       </geometry>
     </collision> -->

File: src/description/urdf/basic_terrain_v2_leaves_001_002.urdf.xacro (robot description, xacro)
@@ -10,5 +10,5 @@
       <origin xyz="0 0 0" rpy="0 0 0" />
       <geometry>
-        <mesh filename="file://$(find custom_gazebo)/src/description/meshes/basic_terrain_v2_leaves_001_002.dae" />
+        <mesh filename="file://$(find custom_gazebo_world)/src/description/meshes/basic_terrain_v2_leaves_001_002.dae" />
       </geometry>
     </visual>
@@ -16,5 +16,5 @@
       <origin xyz="0 0 0" rpy="0 0 0" />
       <geometry>
-        <mesh filename="file://$(find custom_gazebo)/src/description/meshes/basic_terrain_v2_leaves_001_002.dae" />
+        <mesh filename="file://$(find custom_gazebo_world)/src/description/meshes/basic_terrain_v2_leaves_001_002.dae" />
       </geometry>
     </collision> -->

File: src/description/urdf/basic_terrain_v2_leaves_002.urdf.xacro (robot description, xacro)
@@ -10,5 +10,5 @@
       <origin xyz="0 0 0" rpy="0 0 0" />
       <geometry>
-        <mesh filename="file://$(find custom_gazebo)/src/description/meshes/basic_terrain_v2_leaves_002.dae" />
+        <mesh filename="file://$(find custom_gazebo_world)/src/description/meshes/basic_terrain_v2_leaves_002.dae" />
       </geometry>
     </visual>
@@ -16,5 +16,5 @@
       <origin xyz="0 0 0" rpy="0 0 0" />
       <geometry>
-        <mesh filename="file://$(find custom_gazebo)/src/description/meshes/basic_terrain_v2_leaves_002.dae" />
+        <mesh filename="file://$(find custom_gazebo_world)/src/description/meshes/basic_terrain_v2_leaves_002.dae" />
       </geometry>
     </collision> -->

File: src/description/urdf/basic_terrain_v2_tree.urdf.xacro (robot description, xacro)
@@ -10,5 +10,5 @@
       <origin xyz="0 0 0" rpy="0 0 0" />
       <geometry>
-        <mesh filename="file://$(find custom_gazebo)/src/description/meshes/basic_terrain_v2_tree.dae" />
+        <mesh filename="file://$(find custom_gazebo_world)/src/description/meshes/basic_terrain_v2_tree.dae" />
       </geometry>
     </visual>
@@ -16,5 +16,5 @@
       <origin xyz="0 0 0" rpy="0 0 0" />
       <geometry>
-        <mesh filename="file://$(find custom_gazebo)/src/description/meshes/basic_terrain_v2_tree.dae" />
+        <mesh filename="file://$(find custom_gazebo_world)/src/description/meshes/basic_terrain_v2_tree.dae" />
       </geometry>
     </collision>

File: src/description/urdf/basic_terrain_v2_tree_001.urdf.xacro (robot description, xacro)
@@ -10,5 +10,5 @@
       <origin xyz="0 0 0" rpy="0 0 0" />
       <geometry>
-        <mesh filename="file://$(find custom_gazebo)/src/description/meshes/basic_terrain_v2_tree_001.dae" />
+        <mesh filename="file://$(find custom_gazebo_world)/src/description/meshes/basic_terrain_v2_tree_001.dae" />
       </geometry>
     </visual>
@@ -16,5 +16,5 @@
       <origin xyz="0 0 0" rpy="0 0 0" />
       <geometry>
-        <mesh filename="file://$(find custom_gazebo)/src/description/meshes/basic_terrain_v2_tree_001.dae" />
+        <mesh filename="file://$(find custom_gazebo_world)/src/description/meshes/basic_terrain_v2_tree_001.dae" />
       </geometry>
     </collision>

File: src/description/urdf/basic_terrain_v2_tree_001_003.urdf.xacro (robot description, xacro)
@@ -10,5 +10,5 @@
       <origin xyz="0 0 0" rpy="0 0 0" />
       <geometry>
-        <mesh filename="file://$(find custom_gazebo)/src/description/meshes/basic_terrain_v2_tree_001_003.dae" />
+        <mesh filename="file://$(find custom_gazebo_world)/src/description/meshes/basic_terrain_v2_tree_001_003.dae" />
       </geometry>
     </visual>
@@ -16,5 +16,5 @@
       <origin xyz="0 0 0" rpy="0 0 0" />
       <geometry>
-        <mesh filename="file://$(find custom_gazebo)/src/description/meshes/basic_terrain_v2_tree_001_003.dae" />
+        <mesh filename="file://$(find custom_gazebo_world)/src/description/meshes/basic_terrain_v2_tree_001_003.dae" />
       </geometry>
     </collision>

File: src/description/urdf/basic_terrain_v2_tree_002.urdf.xacro (robot description, xacro)
@@ -10,5 +10,5 @@
       <origin xyz="0 0 0" rpy="0 0 0" />
       <geometry>
-        <mesh filename="file://$(find custom_gazebo)/src/description/meshes/basic_terrain_v2_tree_002.dae" />
+        <mesh filename="file://$(find custom_gazebo_world)/src/description/meshes/basic_terrain_v2_tree_002.dae" />
       </geometry>
     </visual>
@@ -16,5 +16,5 @@
       <origin xyz="0 0 0" rpy="0 0 0" />
       <geometry>
-        <mesh filename="file://$(find custom_gazebo)/src/description/meshes/basic_terrain_v2_tree_002.dae" />
+        <mesh filename="file://$(find custom_gazebo_world)/src/description/meshes/basic_terrain_v2_tree_002.dae" />
       </geometry>
     </collision>
