Commit message: changed the package name

File: urdf/basic_terrain_v3_Grass.urdf.xacro (robot description, xacro)
@@ -9,5 +9,5 @@
       <origin xyz="0 0 0" rpy="0 0 0" />
       <geometry>
-        <mesh filename="package://custom_terrain/meshes/basic_terrain_v3_Grass.dae" />
+        <mesh filename="package://custom_gazebo_world/meshes/basic_terrain_v3_Grass.dae" />
       </geometry>
     </visual>
@@ -15,5 +15,5 @@
       <origin xyz="0 0 0" rpy="0 0 0" />
       <geometry>
-        <mesh filename="package://custom_terrain/meshes/basic_terrain_v3_Grass.dae" />
+        <mesh filename="package://custom_gazebo_world/meshes/basic_terrain_v3_Grass.dae" />
       </geometry>
     </collision>

File: urdf/basic_terrain_v3_Grass_001.urdf.xacro (robot description, xacro)
@@ -9,5 +9,5 @@
       <origin xyz="0 0 0" rpy="0 0 0" />
       <geometry>
-        <mesh filename="package://custom_terrain/meshes/basic_terrain_v3_Grass_001.dae" />
+        <mesh filename="package://custom_gazebo_world/meshes/basic_terrain_v3_Grass_001.dae" />
       </geometry>
     </visual>
@@ -15,5 +15,5 @@
       <origin xyz="0 0 0" rpy="0 0 0" />
       <geometry>
-        <mesh filename="package://custom_terrain/meshes/basic_terrain_v3_Grass_001.dae" />
+        <mesh filename="package://custom_gazebo_world/meshes/basic_terrain_v3_Grass_001.dae" />
       </geometry>
     </collision>

File: urdf/basic_terrain_v3_Grass_002.urdf.xacro (robot description, xacro)
@@ -9,5 +9,5 @@
       <origin xyz="0 0 0" rpy="0 0 0" />
       <geometry>
-        <mesh filename="package://custom_terrain/meshes/basic_terrain_v3_Grass_002.dae" />
+        <mesh filename="package://custom_gazebo_world/meshes/basic_terrain_v3_Grass_002.dae" />
       </geometry>
     </visual>
@@ -15,5 +15,5 @@
       <origin xyz="0 0 0" rpy="0 0 0" />
       <geometry>
-        <mesh filename="package://custom_terrain/meshes/basic_terrain_v3_Grass_002.dae" />
+        <mesh filename="package://custom_gazebo_world/meshes/basic_terrain_v3_Grass_002.dae" />
       </geometry>
     </collision> -->

File: urdf/basic_terrain_v3_Landscape_01.urdf.xacro (robot description, xacro)
@@ -9,5 +9,5 @@
       <origin xyz="0 0 0" rpy="0 0 0" />
       <geometry>
-        <mesh filename="package://custom_terrain/meshes/basic_terrain_v3_Landscape_01.dae" />
+        <mesh filename="package://custom_gazebo_world/meshes/basic_terrain_v3_Landscape_01.dae" />
       </geometry>
     </visual>
@@ -15,5 +15,5 @@
       <origin xyz="0 0 0" rpy="0 0 0" />
       <geometry>
-        <mesh filename="package://custom_terrain/meshes/basic_terrain_v3_Landscape_01.dae" />
+        <mesh filename="package://custom_gazebo_world/meshes/basic_terrain_v3_Landscape_01.dae" />
       </geometry>
     </collision>

File: urdf/basic_terrain_v3_leaves.urdf.xacro (robot description, xacro)
@@ -9,5 +9,5 @@
       <origin xyz="0 0 0" rpy="0 0 0" />
       <geometry>
-        <mesh filename="package://custom_terrain/meshes/basic_terrain_v3_leaves.dae" />
+        <mesh filename="package://custom_gazebo_world/meshes/basic_terrain_v3_leaves.dae" />
       </geometry>
     </visual>
@@ -15,5 +15,5 @@
       <origin xyz="0 0 0" rpy="0 0 0" />
       <geometry>
-        <mesh filename="package://custom_terrain/meshes/basic_terrain_v3_leaves.dae" />
+        <mesh filename="package://custom_gazebo_world/meshes/basic_terrain_v3_leaves.dae" />
       </geometry>
     </collision>

File: urdf/basic_terrain_v3_leaves_001.urdf.xacro (robot description, xacro)
@@ -9,5 +9,5 @@
       <origin xyz="0 0 0" rpy="0 0 0" />
       <geometry>
-        <mesh filename="package://custom_terrain/meshes/basic_terrain_v3_leaves_001.dae" />
+        <mesh filename="package://custom_gazebo_world/meshes/basic_terrain_v3_leaves_001.dae" />
       </geometry>
     </visual>
@@ -15,5 +15,5 @@
       <origin xyz="0 0 0" rpy="0 0 0" />
       <geometry>
-        <mesh filename="package://custom_terrain/meshes/basic_terrain_v3_leaves_001.dae" />
+        <mesh filename="package://custom_gazebo_world/meshes/basic_terrain_v3_leaves_001.dae" />
       </geometry>
     </collision>

File: urdf/basic_terrain_v3_leaves_001_001.urdf.xacro (robot description, xacro)
@@ -9,5 +9,5 @@
       <origin xyz="0 0 0" rpy="0 0 0" />
       <geometry>
-        <mesh filename="package://custom_terrain/meshes/basic_terrain_v3_leaves_001_001.dae" />
+        <mesh filename="package://custom_gazebo_world/meshes/basic_terrain_v3_leaves_001_001.dae" />
       </geometry>
     </visual>
@@ -15,5 +15,5 @@
       <origin xyz="0 0 0" rpy="0 0 0" />
       <geometry>
-        <mesh filename="package://custom_terrain/meshes/basic_terrain_v3_leaves_001_001.dae" />
+        <mesh filename="package://custom_gazebo_world/meshes/basic_terrain_v3_leaves_001_001.dae" />
       </geometry>
     </collision>

File: urdf/basic_terrain_v3_leaves_001_002.urdf.xacro (robot description, xacro)
@@ -9,5 +9,5 @@
       <origin xyz="0 0 0" rpy="0 0 0" />
       <geometry>
-        <mesh filename="package://custom_terrain/meshes/basic_terrain_v3_leaves_001_002.dae" />
+        <mesh filename="package://custom_gazebo_world/meshes/basic_terrain_v3_leaves_001_002.dae" />
       </geometry>
     </visual>
@@ -15,5 +15,5 @@
       <origin xyz="0 0 0" rpy="0 0 0" />
       <geometry>
-        <mesh filename="package://custom_terrain/meshes/basic_terrain_v3_leaves_001_002.dae" />
+        <mesh filename="package://custom_gazebo_world/meshes/basic_terrain_v3_leaves_001_002.dae" />
       </geometry>
     </collision>

File: urdf/basic_terrain_v3_leaves_002.urdf.xacro (robot description, xacro)
@@ -9,5 +9,5 @@
       <origin xyz="0 0 0" rpy="0 0 0" />
       <geometry>
-        <mesh filename="package://custom_terrain/meshes/basic_terrain_v3_leaves_002.dae" />
+        <mesh filename="package://custom_gazebo_world/meshes/basic_terrain_v3_leaves_002.dae" />
       </geometry>
     </visual>
@@ -15,5 +15,5 @@
       <origin xyz="0 0 0" rpy="0 0 0" />
       <geometry>
-        <mesh filename="package://custom_terrain/meshes/basic_terrain_v3_leaves_002.dae" />
+        <mesh filename="package://custom_gazebo_world/meshes/basic_terrain_v3_leaves_002.dae" />
       </geometry>
     </collision>

File: urdf/basic_terrain_v3_leaves_003.urdf.xacro (robot description, xacro)
@@ -9,5 +9,5 @@
       <origin xyz="0 0 0" rpy="0 0 0" />
       <geometry>
-        <mesh filename="package://custom_terrain/meshes/basic_terrain_v3_leaves_003.dae" />
+        <mesh filename="package://custom_gazebo_world/meshes/basic_terrain_v3_leaves_003.dae" />
       </geometry>
     </visual>
@@ -15,5 +15,5 @@
       <origin xyz="0 0 0" rpy="0 0 0" />
       <geometry>
-        <mesh filename="package://custom_terrain/meshes/basic_terrain_v3_leaves_003.dae" />
+        <mesh filename="package://custom_gazebo_world/meshes/basic_terrain_v3_leaves_003.dae" />
       </geometry>
     </collision>

File: urdf/basic_terrain_v3_rock_001.urdf.xacro (robot description, xacro)
@@ -9,5 +9,5 @@
       <origin xyz="0 0 0" rpy="0 0 0" />
       <geometry>
-        <mesh filename="package://custom_terrain/meshes/basic_terrain_v3_rock_001.dae" />
+        <mesh filename="package://custom_gazebo_world/meshes/basic_terrain_v3_rock_001.dae" />
       </geometry>
     </visual>
@@ -15,5 +15,5 @@
       <origin xyz="0 0 0" rpy="0 0 0" />
       <geometry>
-        <mesh filename="package://custom_terrain/meshes/basic_terrain_v3_rock_001_collision.stl" />
+        <mesh filename="package://custom_gazebo_world/meshes/basic_terrain_v3_rock_001_collision.stl" />
       </geometry>
     </collision>

File: urdf/basic_terrain_v3_rock_001_001.urdf.xacro (robot description, xacro)
@@ -9,5 +9,5 @@
       <origin xyz="0 0 0" rpy="0 0 0" />
       <geometry>
-        <mesh filename="package://custom_terrain/meshes/basic_terrain_v3_rock_001_001.dae" />
+        <mesh filename="package://custom_gazebo_world/meshes/basic_terrain_v3_rock_001_001.dae" />
       </geometry>
     </visual>
@@ -15,5 +15,5 @@
       <origin xyz="0 0 0" rpy="0 0 0" />
       <geometry>
-        <mesh filename="package://custom_terrain/meshes/basic_terrain_v3_rock_001_001.dae" />
+        <mesh filename="package://custom_gazebo_world/meshes/basic_terrain_v3_rock_001_001.dae" />
       </geometry>
     </collision>

File: urdf/basic_terrain_v3_rock_002.urdf.xacro (robot description, xacro)
@@ -9,5 +9,5 @@
       <origin xyz="0 0 0" rpy="0 0 0" />
       <geometry>
-        <mesh filename="package://custom_terrain/meshes/basic_terrain_v3_rock_002.dae" />
+        <mesh filename="package://custom_gazebo_world/meshes/basic_terrain_v3_rock_002.dae" />
       </geometry>
     </visual>
@@ -15,5 +15,5 @@
       <origin xyz="0 0 0" rpy="0 0 0" />
       <geometry>
-        <mesh filename="package://custom_terrain/meshes/basic_terrain_v3_rock_002_collision.stl" />
+        <mesh filename="package://custom_gazebo_world/meshes/basic_terrain_v3_rock_002_collision.stl" />
       </geometry>
     </collision>

File: urdf/basic_terrain_v3_rock_003.urdf.xacro (robot description, xacro)
@@ -9,5 +9,5 @@
       <origin xyz="0 0 0" rpy="0 0 0" />
       <geometry>
-        <mesh filename="package://custom_terrain/meshes/basic_terrain_v3_rock_003.dae" />
+        <mesh filename="package://custom_gazebo_world/meshes/basic_terrain_v3_rock_003.dae" />
       </geometry>
     </visual>
@@ -15,5 +15,5 @@
       <origin xyz="0 0 0" rpy="0 0 0" />
       <geometry>
-        <mesh filename="package://custom_terrain/meshes/basic_terrain_v3_rock_003_collision.stl" />
+        <mesh filename="package://custom_gazebo_world/meshes/basic_terrain_v3_rock_003_collision.stl" />
       </geometry>
     </collision>

File: urdf/basic_terrain_v3_tree.urdf.xacro (robot description, xacro)
@@ -9,5 +9,5 @@
       <origin xyz="0 0 0" rpy="0 0 0" />
       <geometry>
-        <mesh filename="package://custom_terrain/meshes/basic_terrain_v3_tree.dae" />
+        <mesh filename="package://custom_gazebo_world/meshes/basic_terrain_v3_tree.dae" />
       </geometry>
     </visual>
@@ -15,5 +15,5 @@
       <origin xyz="0 0 0" rpy="0 0 0" />
       <geometry>
-        <mesh filename="package://custom_terrain/meshes/basic_terrain_v3_tree_collision.stl" />
+        <mesh filename="package://custom_gazebo_world/meshes/basic_terrain_v3_tree_collision.stl" />
       </geometry>
     </collision>

File: urdf/basic_terrain_v3_tree_001.urdf.xacro (robot description, xacro)
@@ -9,5 +9,5 @@
       <origin xyz="0 0 0" rpy="0 0 0" />
       <geometry>
-        <mesh filename="package://custom_terrain/meshes/basic_terrain_v3_tree_001.dae" />
+        <mesh filename="package://custom_gazebo_world/meshes/basic_terrain_v3_tree_001.dae" />
       </geometry>
     </visual>
@@ -15,5 +15,5 @@
       <origin xyz="0 0 0" rpy="0 0 0" />
       <geometry>
-        <mesh filename="package://custom_terrain/meshes/basic_terrain_v3_tree_001_collision.stl" />
+        <mesh filename="package://custom_gazebo_world/meshes/basic_terrain_v3_tree_001_collision.stl" />
       </geometry>
     </collision>

File: urdf/basic_terrain_v3_tree_001_001.urdf.xacro (robot description, xacro)
@@ -9,5 +9,5 @@
       <origin xyz="0 0 0" rpy="0 0 0" />
       <geometry>
-        <mesh filename="package://custom_terrain/meshes/basic_terrain_v3_tree_001_001.dae" />
+        <mesh filename="package://custom_gazebo_world/meshes/basic_terrain_v3_tree_001_001.dae" />
       </geometry>
     </visual>
@@ -15,5 +15,5 @@
       <origin xyz="0 0 0" rpy="0 0 0" />
       <geometry>
-        <mesh filename="package://custom_terrain/meshes/basic_terrain_v3_tree_001_001_collision.stl" />
+        <mesh filename="package://custom_gazebo_world/meshes/basic_terrain_v3_tree_001_001_collision.stl" />
       </geometry>
     </collision>

File: urdf/basic_terrain_v3_tree_001_002.urdf.xacro (robot description, xacro)
@@ -9,5 +9,5 @@
       <origin xyz="0 0 0" rpy="0 0 0" />
       <geometry>
-        <mesh filename="package://custom_terrain/meshes/basic_terrain_v3_tree_001_002.dae" />
+        <mesh filename="package://custom_gazebo_world/meshes/basic_terrain_v3_tree_001_002.dae" />
       </geometry>
     </visual>
@@ -15,5 +15,5 @@
       <origin xyz="0 0 0" rpy="0 0 0" />
       <geometry>
-        <mesh filename="package://custom_terrain/meshes/basic_terrain_v3_tree_001_002_collision.stl" />
+        <mesh filename="package://custom_gazebo_world/meshes/basic_terrain_v3_tree_001_002_collision.stl" />
       </geometry>
     </collision>

File: urdf/basic_terrain_v3_tree_001_003.urdf.xacro (robot description, xacro)
@@ -9,5 +9,5 @@
       <origin xyz="0 0 0" rpy="0 0 0" />
       <geometry>
-        <mesh filename="package://custom_terrain/meshes/basic_terrain_v3_tree_001_003.dae" />
+        <mesh filename="package://custom_gazebo_world/meshes/basic_terrain_v3_tree_001_003.dae" />
       </geometry>
     </visual>
@@ -15,5 +15,5 @@
       <origin xyz="0 0 0" rpy="0 0 0" />
       <geometry>
-        <mesh filename="package://custom_terrain/meshes/basic_terrain_v3_tree_001_003_collision.stl" />
+        <mesh filename="package://custom_gazebo_world/meshes/basic_terrain_v3_tree_001_003_collision.stl" />
       </geometry>
     </collision>

File: urdf/basic_terrain_v3_tree_002.urdf.xacro (robot description, xacro)
@@ -9,5 +9,5 @@
       <origin xyz="0 0 0" rpy="0 0 0" />
       <geometry>
-        <mesh filename="package://custom_terrain/meshes/basic_terrain_v3_tree_002.dae" />
+        <mesh filename="package://custom_gazebo_world/meshes/basic_terrain_v3_tree_002.dae" />
       </geometry>
     </visual>
@@ -15,5 +15,5 @@
       <origin xyz="0 0 0" rpy="0 0 0" />
       <geometry>
-        <mesh filename="package://custom_terrain/meshes/basic_terrain_v3_tree_002_collision.stl" />
+        <mesh filename="package://custom_gazebo_world/meshes/basic_terrain_v3_tree_002_collision.stl" />
       </geometry>
     </collision>
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
Commit message: update xacro of grass

File: urdf/basic_terrain_v3_Grass.urdf.xacro (robot description, xacro)
@@ -12,10 +12,10 @@
       </geometry>
     </visual>
-    <collision>
+    <!-- <collision>
       <origin xyz="0 0 0" rpy="0 0 0" />
       <geometry>
         <mesh filename="package://custom_gazebo_world/meshes/basic_terrain_v3_Grass.dae" />
       </geometry>
-    </collision>
+    </collision> -->
   </link>
   <gazebo> <static>true</static></gazebo>

File: urdf/basic_terrain_v3_Grass_001.urdf.xacro (robot description, xacro)
@@ -12,10 +12,10 @@
       </geometry>
     </visual>
-    <collision>
+    <!-- <collision>
       <origin xyz="0 0 0" rpy="0 0 0" />
       <geometry>
         <mesh filename="package://custom_gazebo_world/meshes/basic_terrain_v3_Grass_001.dae" />
       </geometry>
-    </collision>
+    </collision> -->
   </link>
   <gazebo> <static>true</static></gazebo>
