Commit message: added new world

File: world_type/hard_world/urdf/terrain_v6_Grass_001.urdf.xacro (robot description, xacro)
@@ -1,4 +1,4 @@
 <robot name="robot">
-  <link name="easy_world_leaves_link">
+  <link name="terrain_v6_Grass_001_link">
     <inertial>
       <origin xyz="0 0 0" rpy="0 0 0" />
@@ -9,5 +9,5 @@
       <origin xyz="0 0 0" rpy="0 0 0" />
       <geometry>
-        <mesh filename="package://custom_gazebo_world/world_type/easy_world/meshes/easy_world_leaves.dae" />
+        <mesh filename="package://custom_gazebo_world/world_type/hard_world/meshes/terrain_v6_Grass_001.dae" />
       </geometry>
     </visual>
@@ -15,5 +15,5 @@
       <origin xyz="0 0 0" rpy="0 0 0" />
       <geometry>
-        <mesh filename="package://custom_gazebo_world/world_type/easy_world/meshes/easy_world_leaves.dae" />
+        <mesh filename="package://custom_gazebo_world/world_type/hard_world/meshes/terrain_v6_Grass_001.dae" />
       </geometry>
     </collision> -->
